File: Hardware/PCB/MainMicro/MainMicro.kicad_sch (KiCad schematic)
At the start: 28 parts, among them J1 Conn_02x05_Odd_Even, J2 USB_B_Mini, U1 AMS1117-3.3, U2 STM32F091CBTx, U3 FT232RL

Commit message: PCB footprint assignment
Parts:
- removed C12, C13, C3, C4, C5, C6: 100n, Capacitor_SMD:C_0805_2012Metric_Pad1.18x1.45mm_HandSolder, symbol pspice:C
- removed C7: 10n, Capacitor_SMD:C_0805_2012Metric_Pad1.18x1.45mm_HandSolder, symbol pspice:C
- removed C8, C9: 1u, Capacitor_SMD:C_0805_2012Metric_Pad1.18x1.45mm_HandSolder, symbol pspice:C
- removed FerriteBead1: 120R, Inductor_SMD:L_0603_1608Metric_Pad1.05x0.95mm_HandSolder, symbol Device:FerriteBead
- removed R?: 100K, Resistor_SMD:R_0805_2012Metric_Pad1.15x1.40mm_HandSolder, symbol Device:R_US
- added C4, C5, C6, C7, C8, C9: .1uF, Capacitor_SMD:C_0805_2012Metric_Pad1.18x1.45mm_HandSolder, symbol Device:C
- added FB1: Ferrite Bead, Inductor_SMD:L_0805_2012Metric_Pad1.15x1.40mm_HandSolder, symbol Device:Ferrite_Bead_Small
- added J4: Conn_01x05_Male, Connector_JST:JST_EH_B5B-EH-A_1x05_P2.50mm_Vertical, symbol Connector:Conn_01x05_Male
- added J5, J6: Conn_01x06_Male, Connector_JST:JST_EH_B6B-EH-A_1x06_P2.50mm_Vertical, symbol Connector:Conn_01x06_Male
- added Q1, Q2, Q3, Q4, Q5, Q6: BSS138, Package_TO_SOT_SMD:SOT-23, symbol Transistor_FET:BSS138
- added R10, R11, R12, R13, R14, R15, R16, R5, R6, R7, R8, R9: 10k, Resistor_SMD:R_0805_2012Metric_Pad1.20x1.40mm_HandSolder, symbol Device:R
- added R2: 100k, Resistor_SMD:R_0805_2012Metric_Pad1.20x1.40mm_HandSolder, symbol Device:R
- C3: renamed from C?; value C -> 100n; footprint (none) -> Capacitor_SMD:C_0805_2012Metric_Pad1.18x1.45mm_HandSolder
- D3: renamed from D?; footprint (none) -> LED_SMD:LED_0805_2012Metric_Pad1.15x1.40mm_HandSolder
- J1: footprint (none) -> Connector_IDC:IDC-Header_2x05_P2.54mm_Latch_Vertical
- J3: renamed from J?; footprint (none) -> Connector_BarrelJack:BarrelJack_SwitchcraftConxall_RAPC10U_Horizontal
- R3: renamed from R?; footprint (none) -> Resistor_SMD:R_0805_2012Metric_Pad1.20x1.40mm_HandSolder
- R4: renamed from R?; value R -> 5k; footprint (none) -> Resistor_SMD:R_0805_2012Metric_Pad1.20x1.40mm_HandSolder
- SW1: renamed from SW?; footprint (none) -> Button_Switch_SMD:SW_SPST_PTS645
- gave numbers to parts that had none: 1
Connections:
- net +3.3VA: now also U2.9 (VDDA), C9.1, FB1.1
- net +3V3: now also C4.1, C5.1, C6.1, C7.1, C8.1, FB1.2, J4.1 (Pin_1), Q1.1 (G), Q2.1 (G), Q3.1 (G), Q4.1 (G), Q5.1 (G), Q6.1 (G), R10.1, R5.1, R6.1, R7.1, R8.1, R9.1
- net +5V: now also R11.1, R12.1, R13.1, R14.1, R15.1, R16.1
- net BOOT0: now also R2.2
- net GND: now also C10.1, C4.2, C5.2, C6.2, C7.2, C8.2, C9.2, J4.5 (Pin_5), J5.1 (Pin_1), J5.3 (Pin_3), J5.5 (Pin_5), J6.1 (Pin_1), J6.3 (Pin_3), J6.5 (Pin_5), R2.1; no longer C10.2
- net VUSB 5V: now also C10.2; no longer C10.1
- net PA8_GPO: now reaches U2.29 (PA8)
- net PA8_GPO: now also Q1.2 (S), R5.2
- net PA9_GPO: now reaches U2.30 (PA9)
- net PA9_GPO: now also Q2.2 (S), R6.2
- net PA10_GPO: now reaches U2.31 (PA10)
- net PA10_GPO: now also Q4.2 (S), R8.2
- net PA11_GPO: now reaches U2.32 (PA11)
- net PA11_GPO: now also Q5.2 (S), R9.2
- net SPI1_SCK: now reaches U2.39 (PB3)
- net SPI1_SCK: now also J4.4 (Pin_4)
- net SPI1_MISO: now reaches U2.40 (PB4)
- net SPI1_MISO: now also J4.3 (Pin_3)
- net SPI1_MOSI: now reaches U2.41 (PB5)
- net SPI1_MOSI: now also J4.2 (Pin_2)
- net PB7_GPO: now reaches U2.43 (PB7)
- net PB7_GPO: now also Q3.2 (S), R7.2
- net PB8_GPO: now reaches U2.45 (PB8)
- net PB8_GPO: now also Q6.2 (S), R10.2
- net CTS renamed USART2_CTS
- net RTS renamed USART2_RTS
- net RX renamed USART2_RX
- net TX renamed USART2_TX
- new net DIR1+: J5.4 (Pin_4), Q2.3 (D), R12.2
- new net DIR2+: J6.4 (Pin_4), Q5.3 (D), R15.2
- new net EN1+: J5.6 (Pin_6), Q3.3 (D), R13.2
- new net EN2+: J6.6 (Pin_6), Q6.3 (D), R16.2
- new net PUL1+: J5.2 (Pin_2), Q1.3 (D), R11.2
- new net PUL2+: J6.2 (Pin_2), Q4.3 (D), R14.2
Other:
- note added: "600Ohm @ 100MHz .3 Ohm DCR, 500 mA"
- moved on the sheet: C10, D2, D3, J1, J2, J3, R4, U2, U3

Commit message: PCB layout start
Parts:
- removed U2: STM32F091CBTx, Package_QFP:LQFP-48_7x7mm_P0.5mm, symbol MCU_ST_STM32F0:STM32F091CBTx
- added C11, C12: .1u, Capacitor_SMD:C_0805_2012Metric_Pad1.18x1.45mm_HandSolder, symbol Device:C
- added U2: STM32F091RCTx, Package_QFP:LQFP-64_10x10mm_P0.5mm, symbol MCU_ST_STM32F0:STM32F091RCTx
- added U4: MAX7375AXR805, Package_TO_SOT_SMD:SOT-323_SC-70, symbol Oscillator:MAX7375AXR805
Connections:
- net +3.3VA: now also U2.13 (VDDA)
- net +3V3: now also C11.1, C12.1, U2.1 (VBAT), U2.19 (VDD), U2.32 (VDD), U2.48 (VDDIO2), U2.64 (VDD), U4.1 (V+); no longer U3.19 (~{RESET})
- net +5V: now also D2.2 (A), J3.1
- net BOOT0: now also U2.60 (PF11)
- net GND: now also C11.2, C12.2, U2.12 (VSSA), U2.18 (VSS), U2.31 (VSS), U2.47 (VSS), U2.63 (VSS), U4.3 (GND)
- net NRST: now also U3.19 (~{RESET}), U2.7 (NRST)
- net PA10_GPO: now also U2.43 (PA10)
- net PA11_GPO: now also U2.44 (PA11)
- net PA8_GPO: now also U2.41 (PA8)
- net PA9_GPO: now also U2.42 (PA9)
- net PB7_GPO: now also U2.59 (PB7)
- net PB8_GPO: now also U2.61 (PB8)
- net SPI1_MISO: now also U2.56 (PB4)
- net SPI1_MOSI: now also U2.57 (PB5)
- net SPI1_SCK: now also U2.55 (PB3)
- net SWCLK_IN: now also U2.49 (PA14)
- net SWDIO_IN: now also U2.46 (PA13)
- net USART2_CTS: now also U2.14 (PA0)
- net USART2_RTS: now also U2.15 (PA1)
- net USART2_RX: now also U2.17 (PA3)
- net USART2_TX: now also U2.16 (PA2)
- net USB_D-: now reaches J2.2 (D-), U3.16 (USBD-)
- net USB_D+: now reaches J2.3 (D+), U3.15 (USBD+)
- new net 8MHz_OSC_IN: U2.3 (PC14), U2.5 (PF0), U4.2 (CLOCK)
- new net IR_Sensor_IO1: U2.37 (PC6)
- new net IR_Sensor_IO2: U2.38 (PC7)
- no-connect marks 17 -> 18

Commit message: Big PCB changes
Parts:
- removed Q1, Q2, Q3, Q4, Q5, Q6: BSS138, Package_TO_SOT_SMD:SOT-23, symbol Transistor_FET:BSS138
- removed R16: 10k, Resistor_SMD:R_0805_2012Metric_Pad1.20x1.40mm_HandSolder, symbol Device:R
- added C13, C14, C15: .1u, Capacitor_SMD:C_0805_2012Metric_Pad1.18x1.45mm_HandSolder, symbol Device:C
- added H1, H2, H3, H4: MountingHole, MountingHole:MountingHole_2.7mm_M2.5, symbol Mechanical:MountingHole
- added J10, J7, J8, J9: Conn_01x03_Male, Connector_JST:JST_EH_B3B-EH-A_1x03_P2.50mm_Vertical, symbol Connector:Conn_01x03_Male
- added J11, J12: Conn_01x05_Male, Connector_JST:JST_EH_B5B-EH-A_1x05_P2.50mm_Vertical, symbol Connector:Conn_01x05_Male
- added U5: SN74AVC8T245PW, Package_SO:TSSOP-24_4.4x7.8mm_P0.65mm, symbol Logic_LevelTranslator:SN74AVC8T245PW
- J3: footprint Connector_BarrelJack:BarrelJack_SwitchcraftConxall_RAPC10U_Horizontal -> Connector_BarrelJack:BarrelJack_CUI_PJ-102AH_Horizontal
- R10, R11, R12, R13, R14, R15, R5, R6, R7, R8, R9: value 10k -> 10
Connections:
- net +3V3: now also C13.1, U5.1 (VCCA); no longer R10.1, R5.1, R6.1, R7.1, R8.1, R9.1
- net +5V: now also C14.2, C15.2, J10.3 (Pin_3), J11.1 (Pin_1), J11.5 (Pin_5), J12.1 (Pin_1), J12.5 (Pin_5), J7.3 (Pin_3), J8.3 (Pin_3), J9.3 (Pin_3), U5.23 (VCCB), U5.24 (VCCB); no longer D2.2 (A), J3.1, R11.1, R12.1, R13.1, R14.1, R15.1
- net DIR1+: now also U5.20 (B2); no longer R12.2
- net DIR2+: now also U5.17 (B5); no longer R15.2
- net EN1+: now also U5.19 (B3); no longer R13.2
- net EN2+: now also U5.16 (B6)
- net GND: now also C13.2, C14.1, C15.1, J10.2 (Pin_2), J11.2 (Pin_2), J11.4 (Pin_4), J12.2 (Pin_2), J12.4 (Pin_4), J7.2 (Pin_2), J8.2 (Pin_2), J9.2 (Pin_2), U5.11 (GND), U5.12 (GND), U5.13 (GND)
- net IR_Sensor_IO1: now also R14.1
- net IR_Sensor_IO2: now also R15.1
- net PA10_GPO: now also U5.6 (A4); no longer R8.2
- net PA11_GPO: now also U5.7 (A5); no longer R9.2
- net PA8_GPO: now also U5.3 (A1); no longer R5.2
- net PA9_GPO: now also U5.4 (A2); no longer R6.2
- net PB7_GPO: now also U5.5 (A3); no longer R7.2
- net PB8_GPO: now also U5.8 (A6); no longer R10.2
- net PUL1+: now also U5.21 (B1); no longer R11.2
- net PUL2+: now also U5.18 (B4); no longer R14.2
- net SPI1_MISO: now also R7.2; no longer J4.3 (Pin_3)
- net SPI1_MOSI: now also R6.2; no longer J4.2 (Pin_2)
- net SPI1_SCK: now also R5.2; no longer J4.4 (Pin_4)
- net SWCLK_IN: now also R9.1; no longer J1.6 (Pin_6)
- net SWDIO_IN: now also R8.1; no longer J1.2 (Pin_2)
- net Limit_SW1: now reaches U2.40 (PC9)
- net Limit_SW1: now also R10.1
- net Limit_SW2: now reaches U2.51 (PC10)
- net Limit_SW2: now also R11.1
- net Limit_SW3: now reaches U2.52 (PC11)
- net Limit_SW3: now also R12.1
- net Limit_SW4: now reaches U2.53 (PC12)
- net Limit_SW4: now also R13.1
- net PB6_GPO: now reaches U2.58 (PB6)
- net PB6_GPO: now also U5.2 (DIR)
- net PB9_GPO: now reaches U2.62 (PB9)
- net PB9_GPO: now also U5.22 (~{OE})
- net SWIM: no longer names the net of J1.5 (Pin_5)
- new net: J12.3 (Pin_3), R15.2
- new net: J1.2 (Pin_2), R8.2
- new net: J4.2 (Pin_2), R6.1
- new net: J11.3 (Pin_3), R14.2
- new net: J8.1 (Pin_1), R11.2
- new net: J9.1 (Pin_1), R12.2
- new net: J4.4 (Pin_4), R5.1
- new net: J4.3 (Pin_3), R7.1
- new net: D2.2 (A), J3.1
- new net: J1.6 (Pin_6), R9.2
- new net: J10.1 (Pin_1), R13.2
- new net: J7.1 (Pin_1), R10.2
- no-connect marks 18 -> 23
Other:
- note added: "5V --> 3.3V LDO"
- note added: "5V Barrel Jack Interface"
- note added: "7 Segment SPI IO"
- note added: "8MHz OSC"
- note added: "BOOT0 Pullup"
- note added: "Gantry Limit Switch IO"
- note added: "Microcontroller Power Decoupling"
- note added: "Motor Level Stepping IO"
- note added: "Programming Header"
- note added: "Puck IR sensor IO"
- note added: "Reset Switch"
- note added: "USB<-->UART IO"
- moved on the sheet: C1, C11, C2, C3, D1, D2, D3, J1, J3, J4, J5, J6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
