File: Hardware/PCB/Scoreboard/Scoreboard.kicad_sch (KiCad schematic)
At the start: 8 parts

Commit message: Updated PCBs
Parts:
- removed J? (x2): DIN-8, symbol Connector:DIN-8
- added H1, H2, H3, H4: MountingHole, MountingHole:MountingHole_2.2mm_M2, symbol Mechanical:MountingHole
- added J2, J3: Conn_01x08_Male, Connector_PinHeader_2.54mm:PinHeader_1x08_P2.54mm_Vertical, symbol Connector:Conn_01x08_Male
- added U3, U4, U5: MC1413D, Package_SO:SOIC-16_3.9x9.9mm_P1.27mm, symbol Transistor_Array:MC1413D
- J1: renamed from J?; footprint (none) -> Connector_PinSocket_2.54mm:PinSocket_1x05_P2.54mm_Vertical
- U1, U2: renamed from U?; footprint (none) -> 74HC595:SO16
- gave numbers to parts that had none: 3
Connections:
- net GND: now also U3.8 (GND), U4.8 (GND), U5.8 (GND)
- net VCC: now also U3.9 (COM), U4.9 (COM), U5.9 (COM)
- net QB1: now reaches U1.1 (QB)
- net QB1: now also U3.7 (I7)
- net QA1: now reaches U1.15 (QA)
- net QA1: now also U5.1 (I1)
- net QC1: now reaches U1.2 (QC)
- net QC1: now also U3.6 (I6)
- net QD1: now reaches U1.3 (QD)
- net QD1: now also U3.5 (I5)
- net QE1: now reaches U1.4 (QE)
- net QE1: now also U3.4 (I4)
- net QF1: now reaches U1.5 (QF)
- net QF1: now also U3.3 (I3)
- net QG1: now reaches U1.6 (QG)
- net QG1: now also U3.2 (I2)
- net QH1: now reaches U1.7 (QH)
- net QH1: now also U3.1 (I1)
- net QB2: now reaches U2.1 (QB)
- net QB2: now also U4.7 (I7)
- net QA2: now reaches U2.15 (QA)
- net QA2: now also U5.2 (I2)
- net QC2: now reaches U2.2 (QC)
- net QC2: now also U4.6 (I6)
- net QD2: now reaches U2.3 (QD)
- net QD2: now also U4.5 (I5)
- net QE2: now reaches U2.4 (QE)
- net QE2: now also U4.4 (I4)
- net QF2: now reaches U2.5 (QF)
- net QF2: now also U4.3 (I3)
- net QG2: now reaches U2.6 (QG)
- net QG2: now also U4.2 (I2)
- net QH2: now reaches U2.7 (QH)
- net QH2: now also U4.1 (I1)
- new net: J3.2 (Pin_2), U4.10 (O7)
- new net: J3.3 (Pin_3), U4.11 (O6)
- new net: J3.4 (Pin_4), U4.12 (O5)
- new net: J3.5 (Pin_5), U4.13 (O4)
- new net: J3.6 (Pin_6), U4.14 (O3)
- new net: J3.7 (Pin_7), U4.15 (O2)
- new net: J3.8 (Pin_8), U4.16 (O1)
- new net: J2.1 (Pin_1), U5.16 (O1)
- new net: J2.2 (Pin_2), U3.10 (O7)
- new net: J2.3 (Pin_3), U3.11 (O6)
- new net: J2.4 (Pin_4), U3.12 (O5)
- new net: J2.5 (Pin_5), U3.13 (O4)
- new net: J2.6 (Pin_6), U3.14 (O3)
- new net: J2.7 (Pin_7), U3.15 (O2)
- new net: J2.8 (Pin_8), U3.16 (O1)
- new net: J3.1 (Pin_1), U5.15 (O2)
- no-connect marks 0 -> 10
Other:
- note added: "Display Driver"
- note added: "Display Selector"
- note added: "Transistor Array"
